File: PCB/PCB.kicad_sch (KiCad schematic)
At the start: 53 parts, among them J1 Conn_01x05, J2 USB_C_Receptacle_USB2.0_16P, J3 Battery, Q1 2N7002, Q2 2N7002, Q3 AO3401A, SW1 SW_Push, SW2 SW_SPDT, U1 nRF52840_E73-2G4M08S1C, U2 BQ24075RGT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

Commit message: added matrix
Parts:
- added D13, D14, D15, D16: 1N4148WT, Diode_SMD:D_SOD-523, symbol Diode:1N4148WT
- added SW4, SW5, SW6, SW7: MX_SW_HS, PCM_marbastlib-mx:SW_MX_HS_CPG151101S11_1u, symbol PCM_marbastlib-mx:MX_SW_HS
Connections:
- net row1: now reaches U1.18 (P0.04/AIN2)
- net row1: now also D14.1 (K), D16.1 (K)
- net col0: now reaches U1.3 (P0.03/AIN1)
- net col0: now also SW4.1, SW5.1
- net row0: now reaches U1.4 (P0.28/AIN4)
- net row0: now also D13.1 (K), D15.1 (K)
- net col1: now reaches U1.7 (P0.02/AIN0)
- net col1: now also SW6.1, SW7.1
- new net: D16.2 (A), SW7.2
- new net: D14.2 (A), SW5.2
- new net: D15.2 (A), SW6.2
- new net: D13.2 (A), SW4.2
