File: PCB/_autosave-PCB.kicad_pcb (KiCad board)
At the start: 2 copper layers, 10.1 x 6.4 mm, 148 parts, among them J1 USB_C_Receptacle_USB2.0_16P, J2 Battery, J3 Conn_01x04, J4 Conn_01x05, Q1 AO3401A, Q2 2N7002, Q3 2N7002, SW1 SW_Push, SW10 MX_SW_HS, SW11 MX_SW_HS, SW12 MX_SW_HS, SW13 MX_SW_HS, SW14 MX_SW_HS, SW15 MX_SW_HS, SW16 MX_SW_HS, SW17 MX_SW_HS, SW18 MX_SW_HS, SW19 MX_SW_HS, SW2 MX_SW_HS, SW20 MX_SW_HS, SW21 MX_SW_HS, SW22 MX_SW_HS, SW23 MX_SW_HS, SW24 MX_SW_HS, SW25 MX_SW_HS, SW26 MX_SW_HS, SW27 MX_SW_HS, SW28 MX_SW_HS, SW29 MX_SW_HS, SW3 MX_SW_HS, SW30 SW_SPDT, SW31 MX_SW_HS, SW32 MX_SW_HS, SW33 MX_SW_HS, SW34 MX_SW_HS, SW35 MX_SW_HS, SW36 MX_SW_HS, SW37 MX_SW_HS, SW4 MX_SW_HS, SW5 MX_SW_HS, SW6 MX_SW_HS, SW7 MX_SW_HS, SW8 MX_SW_HS, SW9 MX_SW_HS, U1 MAX17048, U2 DW01A, U3 FS8205, U4 BQ24075RGT, U5 nRF52840_E73-2G4M08S1C, Y1 32.768 KHz

Commit message: Tried LEDs, too complicated
Parts:
- moved D30 188.8 mm to (204.8, 54.3)
- moved D31 188.8 mm to (185.7, 54.3)
- moved D29 180.8 mm to (223.8, 54.3)
- moved D32 163.9 mm to (166.6, 54.3)
- moved D33 139.9 mm to (147.6, 54.3)
- moved D34 117.1 mm to (128.5, 54.3)
- moved D28 117.1 mm to (109.5, 73.4)
- moved D21 114.3 mm to (109.5, 92.5)
- moved D7 114.3 mm to (109.5, 130.5)
- moved D1 114.3 mm to (223.8, 130.5)
- moved D15 114.3 mm to (223.8, 92.5)
- moved D35 96.5 mm to (109.5, 54.3)
- moved D27 96.5 mm to (128.6, 73.4)
- moved D20 76.2 mm to (128.6, 92.5)
- moved D2 76.2 mm to (204.8, 130.5)
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Routing:
- net Net-(D22-DOUT): track 0.00 -> 32.9 mm
- net Net-(D15-DIN): track 0.00 -> 32.7 mm
- net Net-(D24-DIN): track 0.00 -> 32.6 mm
- net Net-(D25-DIN): track 0.00 -> 31.6 mm
- net Net-(D13-DIN): track 0.00 -> 31.6 mm
- net Net-(D11-DIN): track 0.00 -> 31.5 mm
- net Net-(D8-DIN): track 0.00 -> 31.3 mm
- net Net-(D23-DIN): track 0.00 -> 31.2 mm
- net Net-(D10-DIN): track 0.00 -> 31.2 mm
- net Net-(D27-DIN): track 0.00 -> 31.1 mm
- net Net-(D12-DIN): track 0.00 -> 31.1 mm
- net Net-(D22-DIN): track 0.00 -> 31.1 mm
- net Net-(D10-DOUT): track 0.00 -> 31.1 mm
- net Net-(D26-DIN): track 0.00 -> 31.1 mm
- net Net-(D14-DIN): track 0.00 -> 22.1 mm
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